File: MiniFanController.brd (EAGLE design)
At the start: 17.8 x 51.4 mm, 23 parts, among them J1 MOLEX_47053-1000MOLEX_47053-1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, J2 MOLEX_47053-1000MOLEX_47053-1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, J3 MOLEX_47053-1000MOLEX_47053-1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, J5 TSW-102-07-G-S, Q1 MICRO_COMMERCIAL_MMSS8050-L-T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, Q2 DIODES_INC_DMP3099L-13DIODES_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, Q3 MICRO_COMMERCIAL_MMSS8050-L-T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, Q4 MICRO_COMMERCIAL_MMSS8050-L-T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, Q5 DIODES_INC_DMP3099L-13DIODES_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, Q6 MICRO_COMMERCIAL_MMSS8050-L-T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, U1 NANO_FOOTPRINT

Commit message: v2 commit. Added current limiting base resistors (oops)
Parts:
- added R12, R13, R14, R15: 2.2k, rcl:R0603
- moved R5 13.0 mm to (7.14, 7.30), turned to 180 degrees
- moved R4 3.18 mm to (6.99, 25.4)
- moved R9 3.18 mm to (6.99, 22.9)
Connections:
- new net N$3: Q1.1, R12.2, R5.2
- new net N$4: Q4.1, R10.2, R13.2
- new net N$5: Q3.1, R14.2, R4.2
- new net N$6: Q6.1, R15.2, R9.2
- net 12V_EN1: now also R14.1; no longer Q3.1, R4.2
- net 12V_EN2: now also R15.1; no longer Q6.1, R9.2
- net PWM1: now also R12.1; no longer Q1.1, R5.2
- net PWM2: now also R13.1; no longer Q4.1, R10.2
Routing:
- net 12V_EN1: track 25.2 -> 1.69 mm, vias 2 -> 0
- net N$5: track 0.00 -> 21.7 mm, vias 0 -> 2
- net N$4: track 0.00 -> 14.4 mm, vias 0 -> 2
- net PWM2: track 21.5 -> 7.67 mm, vias 2 -> 0
- net 12V_EN2: track 15.1 -> 1.69 mm, vias 2 -> 0
- net N$6: track 0.00 -> 11.8 mm, vias 0 -> 2
- net N$3: track 0.00 -> 4.26 mm
- net PWM_FAN1: track 25.3 -> 28.4 mm
- net GND: track 15.3 -> 18.1 mm
- net N$2: track 7.56 -> 6.29 mm
- net PWM1: track 11.1 -> 12.1 mm, vias 0 -> 1
Other:
- board text added: "+"
- board text added: "-"
- board text added: "P"
- board text added: "T"
- board text added: "v2"

Commit message: Fix PMOS Source-Drain mixup
Connections:
- net +12V: now also Q2.2, Q5.2; no longer Q2.3, Q5.3
- net 12V_FAN1: now also Q2.3; no longer Q2.2
- net 12V_FAN2: now also Q5.3; no longer Q5.2
Routing:
- net PWM_FAN1: track 28.4 -> 25.3 mm
- net 12V_FAN1: track 6.15 -> 3.92 mm
- net 12V_FAN2: track 6.47 -> 4.24 mm
- net +12V: track 58.9 -> 61.1 mm, vias 3 -> 2
- net PWM_FAN2: track 46.4 -> 45.1 mm
- net PWM1: track 12.1 -> 11.2 mm
- net GND: track 18.1 -> 17.5 mm, vias 31 -> 35
- net +3V3: track 11.0 -> 10.5 mm
