File: MiniFanController.sch (EAGLE design)
At the start: 23 parts, among them J1 MOLEX_47053-1000MOLEX_47053-1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, J2 MOLEX_47053-1000MOLEX_47053-1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, J3 MOLEX_47053-1000MOLEX_47053-1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, J5 TSW-102-07-G-S, Q1 MICRO_COMMERCIAL_MMSS8050-L-T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, Q2 DIODES_INC_DMP3099L-13DIODES_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, Q3 MICRO_COMMERCIAL_MMSS8050-L-T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, Q4 MICRO_COMMERCIAL_MMSS8050-L-T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, Q5 DIODES_INC_DMP3099L-13DIODES_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, Q6 MICRO_COMMERCIAL_MMSS8050-L-T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, U1 NANO_FOOTPRINT

Commit message: v2 commit. Added current limiting base resistors (oops)
Parts:
- added R12, R13, R14, R15: 2.2k, rcl:R-US_R0603
Connections:
- new net N$3: Q1.B, R12.2, R5.2
- new net N$4: Q4.B, R10.2, R13.2
- new net N$5: Q3.B, R14.2, R4.2
- new net N$6: Q6.B, R15.2, R9.2
- net 12V_EN1: now also R14.1; no longer Q3.B, R4.2
- net 12V_EN2: now also R15.1; no longer Q6.B, R9.2
- net PWM1: now also R12.1; no longer Q1.B, R5.2
- net PWM2: now also R13.1; no longer Q4.B, R10.2
Other:
- moved on the sheet: Q2, Q3, Q5, Q6, R3, R4, R8, R9

Commit message: Fix PMOS Source-Drain mixup
Connections:
- net +12V: now also Q2.S, Q5.S; no longer Q2.D, Q5.D
- net 12V_FAN1: now also Q2.D; no longer Q2.S
- net 12V_FAN2: now also Q5.D; no longer Q5.S
Other:
- moved on the sheet: Q2, Q5
Changed lines of the file:
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@@
 <attribute name="VALUE" x="104.14" y="-40.64" size="1.778" layer="96" rot="R90"/>
 </instance>
-<instance part="Q2" gate="G$0" x="210.82" y="-48.26" smashed="yes">
-<attribute name="NAME" x="221.742" y="-50.8" size="2.54" layer="95" align="top-left"/>
+<instance part="Q2" gate="G$0" x="210.82" y="-58.42" smashed="yes" rot="MR180">
+<attribute name="NAME" x="221.742" y="-55.88" size="2.54" layer="95" rot="MR180" align="top-left"/>
 </instance>
 <instance part="P+4" gate="1" x="215.9" y="-33.02" smashed="yes">
@@
 <attribute name="VALUE" x="104.14" y="-99.06" size="1.778" layer="96" rot="R90"/>
 </instance>
-<instance part="Q5" gate="G$0" x="210.82" y="-106.68" smashed="yes">
-<attribute name="NAME" x="221.742" y="-109.22" size="2.54" layer="95" align="top-left"/>
+<instance part="Q5" gate="G$0" x="210.82" y="-116.84" smashed="yes" rot="MR180">
+<attribute name="NAME" x="221.742" y="-114.3" size="2.54" layer="95" rot="MR180" align="top-left"/>
 </instance>
 <instance part="P+6" gate="1" x="215.9" y="-91.44" smashed="yes">
@@
 </segment>
 <segment>
-<pinref part="Q2" gate="G$0" pin="D"/>
 <pinref part="P+4" gate="1" pin="+12V"/>
 <wire x1="215.9" y1="-35.56" x2="215.9" y2="-38.1" width="0.1524" layer="91"/>
 <pinref part="R3" gate="G$1" pin="2"/>
-<wire x1="215.9" y1="-38.1" x2="215.9" y2="-45.72" width="0.1524" layer="91"/>
 <wire x1="200.66" y1="-40.64" x2="200.66" y2="-38.1" width="0.1524" layer="91"/>
 <wire x1="200.66" y1="-38.1" x2="215.9" y2="-38.1" width="0.1524" layer="91"/>
+<pinref part="Q2" gate="G$0" pin="S"/>
+<wire x1="215.9" y1="-48.26" x2="215.9" y2="-38.1" width="0.1524" layer="91"/>
 <junction x="215.9" y="-38.1"/>
 </segment>
 <segment>
-<pinref part="Q5" gate="G$0" pin="D"/>
 <pinref part="P+6" gate="1" pin="+12V"/>
 <wire x1="215.9" y1="-93.98" x2="215.9" y2="-96.52" width="0.1524" layer="91"/>
 <pinref part="R8" gate="G$1" pin="2"/>
-<wire x1="215.9" y1="-96.52" x2="215.9" y2="-104.14" width="0.1524" layer="91"/>
 <wire x1="200.66" y1="-99.06" x2="200.66" y2="-96.52" width="0.1524" layer="91"/>
 <wire x1="200.66" y1="-96.52" x2="215.9" y2="-96.52" width="0.1524" layer="91"/>
+<pinref part="Q5" gate="G$0" pin="S"/>
+<wire x1="215.9" y1="-106.68" x2="215.9" y2="-96.52" width="0.1524" layer="91"/>
 <junction x="215.9" y="-96.52"/>
 </segment>
@@
 </segment>
 <segment>
-<pinref part="Q5" gate="G$0" pin="S"/>
-<wire x1="215.9" y1="-116.84" x2="215.9" y2="-119.38" width="0.1524" layer="91"/>
-<wire x1="215.9" y1="-119.38" x2="238.76" y2="-119.38" width="0.1524" layer="91"/>
-<label x="220.98" y="-119.38" size="1.778" layer="95"/>
+<wire x1="215.9" y1="-121.92" x2="238.76" y2="-121.92" width="0.1524" layer="91"/>
+<label x="220.98" y="-121.92" size="1.778" layer="95"/>
+<pinref part="Q5" gate="G$0" pin="D"/>
+<wire x1="215.9" y1="-119.38" x2="215.9" y2="-121.92" width="0.1524" layer="91"/>
 </segment>
 </net>
@@
 </segment>
 <segment>
-<pinref part="Q2" gate="G$0" pin="S"/>
-<wire x1="215.9" y1="-58.42" x2="215.9" y2="-60.96" width="0.1524" layer="91"/>
-<wire x1="215.9" y1="-60.96" x2="238.76" y2="-60.96" width="0.1524" layer="91"/>
-<label x="220.98" y="-60.96" size="1.778" layer="95"/>
-</segment>
-</net>
+<wire x1="215.9" y1="-63.5" x2="238.76" y2="-63.5" width="0.1524" layer="91"/>
+<label x="220.98" y="-63.5" size="1.778" layer="95"/>
+<pinref part="Q2" gate="G$0" pin="D"/>
+<wire x1="215.9" y1="-60.96" x2="215.9" y2="-63.5" width="0.1524" layer="91"/>
+</segment>
+</net>
